File: src/pcb/PCB_CircuitAnalyzer/PCB_CircuitAnalyzer.kicad_sch (KiCad schematic)
At the start: 0 parts

Commit message: test
Parts:
- added U1: 74AHC240, symbol 74xx:74AHC240
Changed lines of the file:
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@@
 	(generator_version "9.0")
 	(paper "A4")
+	(symbol
+		(lib_id "74xx:74AHC240")
+		(at 96.52 87.63 0)
+		(unit 1)
+		(exclude_from_sim no)
+		(in_bom yes)
+		(on_board yes)
+		(dnp no)
+		(fields_autoplaced yes)
+		(property "Reference" "U1"
+			(at 98.6633 67.31 0)
+			(effects
+				(font
+					(size 1.27 1.27)
+				)
+				(justify left)
+			)
+		)
+		(property "Value" "74AHC240"
+			(at 98.6633 69.85 0)
+			(effects
+				(font
+					(size 1.27 1.27)
+				)
+				(justify left)
+			)
+		)
+		(property "Footprint" ""
+			(at 96.52 87.63 0)
+			(effects
+				(font
+					(size 1.27 1.27)
+				)
+				(hide yes)
+			)
+		)
+		(property "Datasheet" "https://www.ti.com/lit/ds/symlink/sn54ahc240.pdf"
+			(at 96.52 87.63 0)
+			(effects
+				(font
+					(size 1.27 1.27)
+				)
+				(hide yes)
+			)
+		)
+		(property "Description" "8-bit Buffer/Line Driver 3-state Inverting"
+			(at 96.52 87.63 0)
+			(effects
+				(font
+					(size 1.27 1.27)
+				)
+				(hide yes)
+			)
+		)
+		(pin "13"
+		)
+		(pin "12"
+		)
+		(pin "9"
+		)
+		(pin "5"
+		)
+		(pin "1"
+		)
+		(pin "19"
+		)
+		(pin "14"
+		)
+		(pin "4"
+		)
+		(pin "17"
+		)
+		(pin "10"
+		)
+		(pin "7"
+		)
+		(pin "11"
+		)
+		(pin "2"
+		)
+		(pin "20"
+		)
+		(pin "16"
+		)
+		(pin "15"
+		)
+		(pin "8"
+		)
+		(pin "6"
+		)
+		(pin "18"
+		)
+		(pin "3"
+		)
+		(instances
+			(project ""
+				(path "/54cd8298-f77b-46b8-88fc-3ea0769550b1"
+					(reference "U1")
+					(unit 1)
+				)
+			)
+		)
+	)
 	(sheet_instances
 		(path "/"
